Commit message: fix wrong bringup folder search in xacro

File: src/depthai_ros_driver/urdf/depthai_descr.urdf.xacro (robot description, xacro)
@@ -11,5 +11,5 @@
     <xacro:arg name="cam_pitch"     default="0.0" />
     <xacro:arg name="cam_yaw"       default="0.0" />
-    <xacro:include filename="$(find robot100_description)/urdf/depthai_macro.urdf.xacro"/>
+    <xacro:include filename="$(find depthai_ros_driver)/urdf/depthai_macro.urdf.xacro"/>
     <link name="$(arg parent_frame)"/>
     <xacro:depthai_camera camera_name = "$(arg camera_name)" parent = "$(arg parent_frame)" camera_model = "$(arg camera_model)" base_frame = "$(arg base_frame)" cam_pos_x = "$(arg cam_pos_x)" cam_pos_y = "$(arg cam_pos_y)" cam_pos_z = "$(arg cam_pos_z)" cam_roll = "$(arg cam_roll)" cam_pitch = "$(arg cam_pitch)" cam_yaw = "$(arg cam_yaw)"/>

File: src/depthai_ros_driver/urdf/depthai_macro.urdf.xacro (robot description, xacro)
@@ -32,5 +32,5 @@
             <origin xyz="0 0 0" rpy="0 0 0"/>
             <geometry>
-                <mesh filename="package://robot100_desciption/urdf/models/${model}.stl" />
+                <mesh filename="package://depthai_ros_driver/urdf/models/${model}.stl" />
             </geometry>
             <material name="mat">
